File: TKL.kicad_sch (KiCad schematic)
At the start: 21 parts, among them J1 AVR-ISP-6, U1 ATmega32U4-A, U2 PRTR5V0U2X

Commit message: Matrix
Other:
- added sheet matrix (matrix.kicad_sch)
Changed lines of the file:
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@@
+    )
+  )
+  (sheet (at 284.48 207.01) (size 12.7 3.81) (fields_autoplaced)
+    (stroke (width 0.1524) (type solid))
+    (fill (color 0 0 0 0.0000))
+    (property "Sheetname" "matrix" (at 284.48 206.2984 0)
+      (effects (font (size 1.27 1.27)) (justify left bottom))
+    )
+    (property "Sheetfile" "matrix.kicad_sch" (at 284.48 211.4046 0)
+      (effects (font (size 1.27 1.27)) (justify left top))
+    )
+    (instances
+      (project "TKL"
+        (path "/dd1a797b-d482-4fb7-b017-a28c5b5e9224" (page "2"))
+      )
     )
   )
